Commit message: fix IK theta3: ACD + BAC - pi

File: ros2_ws/src/arm_description/urdf/arm.urdf (robot description, URDF)
Before this commit: robot robotic_arm, 3 links, 2 joints
Links:
- link link_2: geometry visual box size=0.058 0.05 0.03; visual cylinder length=0.14 radius=0.01
Joints:
- joint teta_2: limit lower=0 upper=3.1416 effort=1.0 velocity=1.0 -> lower=-1.5708 upper=1.5708 effort=1.0 velocity=1.0

Commit message: Complete URDF with theta3 and gripper joints

File: ros2_ws/src/arm_description/urdf/arm.urdf (robot description, URDF)
Before this commit: robot robotic_arm, 3 links, 2 joints
Links:
- added link link_3; visual cylinder length=0.14 radius=0.01
Joints:
- added joint teta_3: type revolute, parent link_2, child link_3, origin xyz=0.01 -0.05 0.012 rpy=0 0 0, axis 0 1 0, limit lower=-1.5708 upper=1.5708 effort=1.0 velocity=1.0

Commit message: Complete URDF with all joints and links

File: ros2_ws/src/arm_description/urdf/arm.urdf (robot description, URDF)
Before this commit: robot robotic_arm, 4 links, 3 joints
Links:
- added link gripper; visual cylinder length=0.085 radius=0.01
- link link_3: geometry visual box size=0.027 0.06 0.03; visual cylinder length=0.13 radius=0.01
Joints:
- added joint gripper_joint: type fixed, parent link_3, child gripper, origin xyz=0.1335 -0.024 0 rpy=0 0 0
- joint teta_3: limit lower=-1.5708 upper=1.5708 effort=1.0 velocity=1.0 -> lower=0 upper=1.5708 effort=1.0 velocity=1.0; origin xyz=0.01 -0.05 0.012 rpy=0 0 0 -> xyz=0.025 0.05 0.12 rpy=0 0 0
